Commit message: fix: resulting errors, validated that gazebo launches successfully

File: src/hexa_description/urdf/hexapod.urdf.xacro (robot description, xacro)
@@ -37,5 +37,7 @@
   <xacro:property name="femur_length" value="${geom['leg']['femur_length']}"/>
   <xacro:property name="tibia_length" value="${geom['leg']['tibia_length']}"/>
-  <xacro:property name="seg_radius"   value="${geom['leg']['seg_radius']}"/>
+  <xacro:property name="coxa_radius"  value="${geom['leg']['coxa_radius']}"/>
+  <xacro:property name="femur_radius" value="${geom['leg']['femur_radius']}"/>
+  <xacro:property name="tibia_radius" value="${geom['leg']['tibia_radius']}"/>
   <xacro:property name="coxa_mass"    value="${geom['leg']['coxa_mass']}"/>
   <xacro:property name="femur_mass"   value="${geom['leg']['femur_mass']}"/>
@@ -48,4 +50,38 @@
   <material name="body_grey"><color rgba="0.3 0.3 0.3 1.0"/></material>
   <material name="leg_blue"> <color rgba="0.2 0.4 0.8 1.0"/></material>
+  <!-- =====================================================================
+       Inertial macros. Both compute the tensor from mass + dimensions so
+       the YAML stays the only place a number is typed. Declared before
+       any link uses them: xacro requires macro definitions to precede
+       their first use.
+       ===================================================================== -->
+  <!-- Solid cylinder of length L along the link's local +x:
+         ixx = (1/2) m r^2          (about the long axis)
+         iyy = izz = (1/12) m (3r^2 + L^2)
+       COM at the segment midpoint. -->
+  <xacro:macro name="cylinder_inertial" params="mass length radius">
+    <inertial>
+      <origin xyz="${length/2} 0 0" rpy="0 0 0"/>
+      <mass value="${mass}"/>
+      <inertia ixx="${0.5 * mass * radius * radius}"
+               iyy="${mass * (3*radius*radius + length*length) / 12.0}"
+               izz="${mass * (3*radius*radius + length*length) / 12.0}"
+               ixy="0" ixz="0" iyz="0"/>
+    </inertial>
+  </xacro:macro>
+  <!-- Solid box of side lengths (x, y, z):
+         ixx = (1/12) m (y^2 + z^2)
+         iyy = (1/12) m (x^2 + z^2)
+         izz = (1/12) m (x^2 + y^2)
+       COM at link origin (the body box is centred on base_link). -->
+  <xacro:macro name="box_inertial" params="mass x y z">
+    <inertial>
+      <mass value="${mass}"/>
+      <inertia ixx="${mass * (y*y + z*z) / 12.0}"
+               iyy="${mass * (x*x + z*z) / 12.0}"
+               izz="${mass * (x*x + y*y) / 12.0}"
+               ixy="0" ixz="0" iyz="0"/>
+    </inertial>
+  </xacro:macro>
   <!-- =====================================================================
        Body link — the central chassis everything else hangs off of.
@@ -69,36 +105,4 @@
   </link>
   <!-- =====================================================================
-       Inertial macros. Both compute the tensor from mass + dimensions so
-       the YAML stays the only place a number is typed.
-       ===================================================================== -->
-  <!-- Solid cylinder of length L along the link's local +x:
-         ixx = (1/2) m r^2          (about the long axis)
-         iyy = izz = (1/12) m (3r^2 + L^2)
-       COM at the segment midpoint. -->
-  <xacro:macro name="cylinder_inertial" params="mass length radius">
-    <inertial>
-      <origin xyz="${length/2} 0 0" rpy="0 0 0"/>
-      <mass value="${mass}"/>
-      <inertia ixx="${0.5 * mass * radius * radius}"
-               iyy="${mass * (3*radius*radius + length*length) / 12.0}"
-               izz="${mass * (3*radius*radius + length*length) / 12.0}"
-               ixy="0" ixz="0" iyz="0"/>
-    </inertial>
-  </xacro:macro>
-  <!-- Solid box of side lengths (x, y, z):
-         ixx = (1/12) m (y^2 + z^2)
-         iyy = (1/12) m (x^2 + z^2)
-         izz = (1/12) m (x^2 + y^2)
-       COM at link origin (the body box is centred on base_link). -->
-  <xacro:macro name="box_inertial" params="mass x y z">
-    <inertial>
-      <mass value="${mass}"/>
-      <inertia ixx="${mass * (y*y + z*z) / 12.0}"
-               iyy="${mass * (x*x + z*z) / 12.0}"
-               izz="${mass * (x*x + y*y) / 12.0}"
-               ixy="0" ixz="0" iyz="0"/>
-    </inertial>
-  </xacro:macro>
-  <!-- =====================================================================
        Leg macro.
        Parameters:
@@ -112,5 +116,5 @@
        ===================================================================== -->
   <xacro:macro name="leg" params="side name mount_x mount_y mount_yaw">
-    <!-- ---- Coxa: short horizontal segment attached to the body. -------- -->
+    <!-- Coxa: short horizontal segment attached to the body. -->
     <joint name="${side}_${name}_coxa_joint" type="revolute">
       <parent link="base_link"/>
@@ -130,5 +134,5 @@
         <origin xyz="${coxa_length/2} 0 0" rpy="0 ${pi/2} 0"/>
         <geometry>
-          <cylinder radius="${seg_radius}" length="${coxa_length}"/>
+          <cylinder radius="${coxa_radius}" length="${coxa_length}"/>
         </geometry>
         <material name="leg_blue"/>
@@ -137,12 +141,12 @@
         <origin xyz="${coxa_length/2} 0 0" rpy="0 ${pi/2} 0"/>
         <geometry>
-          <cylinder radius="${seg_radius}" length="${coxa_length}"/>
+          <cylinder radius="${coxa_radius}" length="${coxa_length}"/>
         </geometry>
       </collision>
       <xacro:cylinder_inertial mass="${coxa_mass}"
                                length="${coxa_length}"
-                               radius="${seg_radius}"/>
+                               radius="${coxa_radius}"/>
     </link>
-    <!-- ---- Femur: upper leg, lifts the knee up/down. ------------------- -->
+    <!-- Femur: upper leg, lifts the knee up/down. -->
     <joint name="${side}_${name}_femur_joint" type="revolute">
       <parent link="${side}_${name}_coxa"/>
@@ -161,5 +165,5 @@
         <origin xyz="${femur_length/2} 0 0" rpy="0 ${pi/2} 0"/>
         <geometry>
-          <cylinder radius="${seg_radius}" length="${femur_length}"/>
+          <cylinder radius="${femur_radius}" length="${femur_length}"/>
         </geometry>
         <material name="leg_blue"/>
@@ -168,12 +172,12 @@
         <origin xyz="${femur_length/2} 0 0" rpy="0 ${pi/2} 0"/>
         <geometry>
-          <cylinder radius="${seg_radius}" length="${femur_length}"/>
+          <cylinder radius="${femur_radius}" length="${femur_length}"/>
         </geometry>
       </collision>
       <xacro:cylinder_inertial mass="${femur_mass}"
                                length="${femur_length}"
-                               radius="${seg_radius}"/>
+                               radius="${femur_radius}"/>
     </link>
-    <!-- ---- Tibia: lower leg, bends at the knee down to the foot. ------- -->
+    <!-- Tibia: lower leg, bends at the knee down to the foot. -->
     <joint name="${side}_${name}_tibia_joint" type="revolute">
       <parent link="${side}_${name}_femur"/>
@@ -190,5 +194,5 @@
         <origin xyz="${tibia_length/2} 0 0" rpy="0 ${pi/2} 0"/>
         <geometry>
-          <cylinder radius="${seg_radius}" length="${tibia_length}"/>
+          <cylinder radius="${tibia_radius}" length="${tibia_length}"/>
         </geometry>
         <material name="leg_blue"/>
@@ -197,27 +201,36 @@
         <origin xyz="${tibia_length/2} 0 0" rpy="0 ${pi/2} 0"/>
         <geometry>
-          <cylinder radius="${seg_radius}" length="${tibia_length}"/>
+          <cylinder radius="${tibia_radius}" length="${tibia_length}"/>
         </geometry>
       </collision>
       <xacro:cylinder_inertial mass="${tibia_mass}"
                                length="${tibia_length}"
-                               radius="${seg_radius}"/>
+                               radius="${tibia_radius}"/>
     </link>
-    <!-- ---- Foot: a small sphere at the tip of the tibia. --------------- -->
-    <!-- Used as the IK target and as the ground-contact body in sim. -->
+    <!-- Foot: a small sphere at the tip of the tibia.
+         Used as the IK target and as the ground-contact body in sim.
+         The foot link origin sits at the bottom of the sphere along the
+         tibia's +x axis, so the IK target coincides with the ground
+         contact point under the assumption that the tibia is vertical
+         at touchdown. The sphere geometry is therefore shifted back by
+         -foot_radius in the foot frame to keep its centre at the
+         physical tibia tip. -->
     <joint name="${side}_${name}_foot_joint" type="fixed">
       <parent link="${side}_${name}_tibia"/>
       <child  link="${side}_${name}_foot"/>
-      <origin xyz="${tibia_length} 0 0" rpy="0 0 0"/>
+      <origin xyz="${tibia_length + foot_radius} 0 0" rpy="0 0 0"/>
     </joint>
     <link name="${side}_${name}_foot">
       <visual>
+        <origin xyz="${-foot_radius} 0 0" rpy="0 0 0"/>
         <geometry><sphere radius="${foot_radius}"/></geometry>
         <material name="leg_blue"/>
       </visual>
       <collision>
+        <origin xyz="${-foot_radius} 0 0" rpy="0 0 0"/>
         <geometry><sphere radius="${foot_radius}"/></geometry>
       </collision>
       <inertial>
+        <origin xyz="${-foot_radius} 0 0" rpy="0 0 0"/>
         <mass value="${foot_mass}"/>
         <!-- Solid sphere: I = (2/5) m r^2, isotropic. -->

Commit message: feat: add servo params and differentiate front legs

File: src/hexa_description/urdf/hexapod.urdf.xacro (robot description, xacro)
@@ -77,4 +77,5 @@
   <material name="body_grey"><color rgba="0.3 0.3 0.3 1.0"/></material>
   <material name="leg_blue"> <color rgba="0.2 0.4 0.8 1.0"/></material>
+  <material name="leg_red">  <color rgba="0.8 0.2 0.2 1.0"/></material>
   <!-- =====================================================================
        Inertial macros. Both compute the tensor from mass + dimensions so
@@ -143,4 +144,6 @@
        ===================================================================== -->
   <xacro:macro name="leg" params="side name mount_x mount_y mount_yaw">
+    <!-- Front legs are red to mark orientation; others stay blue. -->
+    <xacro:property name="leg_material" value="${'leg_red' if name == 'front' else 'leg_blue'}"/>
     <!-- Coxa: short horizontal segment attached to the body. -->
     <joint name="${side}_${name}_coxa_joint" type="revolute">
@@ -163,5 +166,5 @@
           <cylinder radius="${coxa_radius}" length="${coxa_length}"/>
         </geometry>
-        <material name="leg_blue"/>
+        <material name="${leg_material}"/>
       </visual>
       <!-- Joint caps: visual-only spheres at each end of the segment. -->
@@ -169,10 +172,10 @@
         <origin xyz="0 0 0" rpy="0 0 0"/>
         <geometry><sphere radius="${coxa_radius}"/></geometry>
-        <material name="leg_blue"/>
+        <material name="${leg_material}"/>
       </visual>
       <visual>
         <origin xyz="${coxa_length} 0 0" rpy="0 0 0"/>
         <geometry><sphere radius="${coxa_radius}"/></geometry>
-        <material name="leg_blue"/>
+        <material name="${leg_material}"/>
       </visual>
       <collision>
@@ -205,15 +208,15 @@
           <cylinder radius="${femur_radius}" length="${femur_length}"/>
         </geometry>
-        <material name="leg_blue"/>
+        <material name="${leg_material}"/>
       </visual>
       <visual>
         <origin xyz="0 0 0" rpy="0 0 0"/>
         <geometry><sphere radius="${femur_radius}"/></geometry>
-        <material name="leg_blue"/>
+        <material name="${leg_material}"/>
       </visual>
       <visual>
         <origin xyz="${femur_length} 0 0" rpy="0 0 0"/>
         <geometry><sphere radius="${femur_radius}"/></geometry>
-        <material name="leg_blue"/>
+        <material name="${leg_material}"/>
       </visual>
       <collision>
@@ -244,5 +247,5 @@
           <cylinder radius="${tibia_radius}" length="${tibia_length}"/>
         </geometry>
-        <material name="leg_blue"/>
+        <material name="${leg_material}"/>
       </visual>
       <!-- Proximal joint cap only; distal end is covered by the foot sphere. -->
@@ -250,5 +253,5 @@
         <origin xyz="0 0 0" rpy="0 0 0"/>
         <geometry><sphere radius="${tibia_radius}"/></geometry>
-        <material name="leg_blue"/>
+        <material name="${leg_material}"/>
       </visual>
       <collision>
@@ -279,5 +282,5 @@
         <origin xyz="${-foot_radius} 0 0" rpy="0 0 0"/>
         <geometry><sphere radius="${foot_radius}"/></geometry>
-        <material name="leg_blue"/>
+        <material name="${leg_material}"/>
       </visual>
       <collision>
