Commit message: feat: default standing posture yaml, consolidate hexa description

File: src/hexa_description/urdf/hexapod.gazebo.xacro (robot description, xacro)
@@ -37,6 +37,6 @@
   <xacro:macro name="foot_contact" params="link">
     <gazebo reference="${link}">
-      <mu1>1.2</mu1>
-      <mu2>1.2</mu2>
+      <mu1>2.0</mu1>
+      <mu2>2.0</mu2>
       <kp>1.0e6</kp>
       <kd>10.0</kd>

File: src/hexa_description/urdf/hexapod.urdf.xacro (robot description, xacro)
@@ -25,9 +25,7 @@
   <!-- =====================================================================
        Config. Geometry (body/leg/foot dimensions, masses, per-leg mounts)
-       and joint limits live in YAML so they can be tuned without editing
-       the URDF. Both files are loaded into Python dicts here.
-       ===================================================================== -->
-  <xacro:property name="joint_limits"
-                  value="${xacro.load_yaml('$(find hexa_description)/config/joint_limits.yaml')}"/>
+       and per-joint-type servo limits live together in geometry.yaml so
+       they can be tuned without editing the URDF.
+       ===================================================================== -->
   <xacro:property name="geom"
                   value="${xacro.load_yaml('$(find hexa_description)/config/geometry.yaml')}"/>
@@ -45,4 +43,33 @@
   <xacro:property name="foot_radius"  value="${geom['foot']['radius']}"/>
   <xacro:property name="foot_mass"    value="${geom['foot']['mass']}"/>
+  <!-- Per-joint <limit> windows, in URDF-convention radians. The YAML
+       carries intuitive per-joint degrees (coxa.deg,
+       femur.above_horizontal_deg, tibia.interior_deg with absolute
+       lower_limit_deg / upper_limit_deg); the conversions here match
+       hexa_kinematics/hexa_kinematics/joint_config.py exactly. The URDF
+       itself stays a pure mathematical presentation of the hexapod —
+       joint zero remains "legs splayed horizontally"; only the <limit>
+       window is shifted to express the servo's reachable range.
+       Sign-aware swap: femur uses -radians(deg) and tibia uses
+       pi - radians(deg), both monotonically decreasing — so intuitive
+       upper_limit_deg maps to URDF lower_rad and vice versa. -->
+  <xacro:property name="coxa_lower_rad"
+                  value="${geom['joints']['coxa']['lower_limit_deg'] * pi / 180}"/>
+  <xacro:property name="coxa_upper_rad"
+                  value="${geom['joints']['coxa']['upper_limit_deg'] * pi / 180}"/>
+  <xacro:property name="femur_lower_rad"
+                  value="${-geom['joints']['femur']['upper_limit_deg'] * pi / 180}"/>
+  <xacro:property name="femur_upper_rad"
+                  value="${-geom['joints']['femur']['lower_limit_deg'] * pi / 180}"/>
+  <xacro:property name="tibia_lower_rad"
+                  value="${pi - geom['joints']['tibia']['upper_limit_deg'] * pi / 180}"/>
+  <xacro:property name="tibia_upper_rad"
+                  value="${pi - geom['joints']['tibia']['lower_limit_deg'] * pi / 180}"/>
+  <!-- Body length and width are derived from the front and middle mounts
+       so the chassis always extends just past the hips: 10% margin per side. -->
+  <xacro:property name="body_length" value="${2 * geom['mounts']['l_front']['x']  * 1.1}"/>
+  <xacro:property name="body_width"  value="${2 * geom['mounts']['l_middle']['y'] * 1.1}"/>
+  <xacro:property name="body_height" value="${geom['body']['height']}"/>
+  <xacro:property name="body_mass"   value="${geom['body']['mass']}"/>
   <!-- =====================================================================
        Materials (just for colour in RViz / Gazebo).
@@ -90,5 +117,5 @@
     <visual>
       <geometry>
-        <box size="${geom['body']['length']} ${geom['body']['width']} ${geom['body']['height']}"/>
+        <box size="${body_length} ${body_width} ${body_height}"/>
       </geometry>
       <material name="body_grey"/>
@@ -96,11 +123,11 @@
     <collision>
       <geometry>
-        <box size="${geom['body']['length']} ${geom['body']['width']} ${geom['body']['height']}"/>
+        <box size="${body_length} ${body_width} ${body_height}"/>
       </geometry>
     </collision>
-    <xacro:box_inertial mass="${geom['body']['mass']}"
-                        x="${geom['body']['length']}"
-                        y="${geom['body']['width']}"
-                        z="${geom['body']['height']}"/>
+    <xacro:box_inertial mass="${body_mass}"
+                        x="${body_length}"
+                        y="${body_width}"
+                        z="${body_height}"/>
   </link>
   <!-- =====================================================================
@@ -124,8 +151,8 @@
       <!-- Rotates around +z = swings the leg forward/backward. -->
       <axis xyz="0 0 1"/>
-      <limit lower="${joint_limits['coxa']['lower']}"
-             upper="${joint_limits['coxa']['upper']}"
-             effort="${joint_limits['coxa']['effort']}"
-             velocity="${joint_limits['coxa']['velocity']}"/>
+      <limit lower="${coxa_lower_rad}"
+             upper="${coxa_upper_rad}"
+             effort="${geom['joints']['coxa']['effort']}"
+             velocity="${geom['joints']['coxa']['velocity']}"/>
     </joint>
     <link name="${side}_${name}_coxa">
@@ -136,4 +163,15 @@
           <cylinder radius="${coxa_radius}" length="${coxa_length}"/>
         </geometry>
+        <material name="leg_blue"/>
+      </visual>
+      <!-- Joint caps: visual-only spheres at each end of the segment. -->
+      <visual>
+        <origin xyz="0 0 0" rpy="0 0 0"/>
+        <geometry><sphere radius="${coxa_radius}"/></geometry>
+        <material name="leg_blue"/>
+      </visual>
+      <visual>
+        <origin xyz="${coxa_length} 0 0" rpy="0 0 0"/>
+        <geometry><sphere radius="${coxa_radius}"/></geometry>
         <material name="leg_blue"/>
       </visual>
@@ -156,8 +194,8 @@
       <!-- Rotates around the leg's local +y = lifts/lowers the femur. -->
       <axis xyz="0 1 0"/>
-      <limit lower="${joint_limits['femur']['lower']}"
-             upper="${joint_limits['femur']['upper']}"
-             effort="${joint_limits['femur']['effort']}"
-             velocity="${joint_limits['femur']['velocity']}"/>
+      <limit lower="${femur_lower_rad}"
+             upper="${femur_upper_rad}"
+             effort="${geom['joints']['femur']['effort']}"
+             velocity="${geom['joints']['femur']['velocity']}"/>
     </joint>
     <link name="${side}_${name}_femur">
@@ -167,4 +205,14 @@
           <cylinder radius="${femur_radius}" length="${femur_length}"/>
         </geometry>
+        <material name="leg_blue"/>
+      </visual>
+      <visual>
+        <origin xyz="0 0 0" rpy="0 0 0"/>
+        <geometry><sphere radius="${femur_radius}"/></geometry>
+        <material name="leg_blue"/>
+      </visual>
+      <visual>
+        <origin xyz="${femur_length} 0 0" rpy="0 0 0"/>
+        <geometry><sphere radius="${femur_radius}"/></geometry>
         <material name="leg_blue"/>
       </visual>
@@ -185,8 +233,8 @@
       <origin xyz="${femur_length} 0 0" rpy="0 0 0"/>
       <axis xyz="0 1 0"/>
-      <limit lower="${joint_limits['tibia']['lower']}"
-             upper="${joint_limits['tibia']['upper']}"
-             effort="${joint_limits['tibia']['effort']}"
-             velocity="${joint_limits['tibia']['velocity']}"/>
+      <limit lower="${tibia_lower_rad}"
+             upper="${tibia_upper_rad}"
+             effort="${geom['joints']['tibia']['effort']}"
+             velocity="${geom['joints']['tibia']['velocity']}"/>
     </joint>
     <link name="${side}_${name}_tibia">
@@ -196,4 +244,10 @@
           <cylinder radius="${tibia_radius}" length="${tibia_length}"/>
         </geometry>
+        <material name="leg_blue"/>
+      </visual>
+      <!-- Proximal joint cap only; distal end is covered by the foot sphere. -->
+      <visual>
+        <origin xyz="0 0 0" rpy="0 0 0"/>
+        <geometry><sphere radius="${tibia_radius}"/></geometry>
         <material name="leg_blue"/>
       </visual>
@@ -255,5 +309,6 @@
     <!-- Front/rear mirror (only affects rear): flips x, reflects yaw about pi/2. -->
     <xacro:property name="x_after_fr"   value="${-ref['x']   if name == 'rear' else ref['x']}"/>
-    <xacro:property name="yaw_after_fr" value="${pi - ref['yaw'] if name == 'rear' else ref['yaw']}"/>
+    <xacro:property name="ref_yaw"      value="${ref['yaw_deg'] * pi / 180}"/>
+    <xacro:property name="yaw_after_fr" value="${pi - ref_yaw if name == 'rear' else ref_yaw}"/>
     <!-- Left/right mirror (only affects right side): flips y, negates yaw. -->
     <xacro:property name="mx"  value="${x_after_fr}"/>
@@ -280,6 +335,6 @@
     <joint name="${side}_${name}_coxa_joint">
       <command_interface name="position">
-        <param name="min">${joint_limits['coxa']['lower']}</param>
-        <param name="max">${joint_limits['coxa']['upper']}</param>
+        <param name="min">${coxa_lower_rad}</param>
+        <param name="max">${coxa_upper_rad}</param>
       </command_interface>
       <state_interface name="position"/>
@@ -288,6 +343,6 @@
     <joint name="${side}_${name}_femur_joint">
       <command_interface name="position">
-        <param name="min">${joint_limits['femur']['lower']}</param>
-        <param name="max">${joint_limits['femur']['upper']}</param>
+        <param name="min">${femur_lower_rad}</param>
+        <param name="max">${femur_upper_rad}</param>
       </command_interface>
       <state_interface name="position"/>
@@ -296,6 +351,6 @@
     <joint name="${side}_${name}_tibia_joint">
       <command_interface name="position">
-        <param name="min">${joint_limits['tibia']['lower']}</param>
-        <param name="max">${joint_limits['tibia']['upper']}</param>
+        <param name="min">${tibia_lower_rad}</param>
+        <param name="max">${tibia_upper_rad}</param>
       </command_interface>
       <state_interface name="position"/>

Commit message: feat: make urdf front legs red

File: src/hexa_description/urdf/hexapod.gazebo.xacro (robot description, xacro)
@@ -20,7 +20,8 @@
   </gazebo>
   <xacro:macro name="leg_material" params="side name">
-    <gazebo reference="${side}_${name}_coxa"> <material>Gazebo/Blue</material></gazebo>
-    <gazebo reference="${side}_${name}_femur"><material>Gazebo/Blue</material></gazebo>
-    <gazebo reference="${side}_${name}_tibia"><material>Gazebo/Blue</material></gazebo>
+    <xacro:property name="gz_colour" value="${'Gazebo/Red' if name == 'front' else 'Gazebo/Blue'}"/>
+    <gazebo reference="${side}_${name}_coxa"> <material>${gz_colour}</material></gazebo>
+    <gazebo reference="${side}_${name}_femur"><material>${gz_colour}</material></gazebo>
+    <gazebo reference="${side}_${name}_tibia"><material>${gz_colour}</material></gazebo>
   </xacro:macro>
   <xacro:leg_material side="l" name="front"/>

Commit message: feat: add initialize and fold phases to hexa_gait

File: src/hexa_description/urdf/hexapod.gazebo.xacro (robot description, xacro)
@@ -18,4 +18,7 @@
   <gazebo reference="base_link">
     <material>Gazebo/DarkGrey</material>
+  </gazebo>
+  <gazebo reference="middle_bar">
+    <material>Gazebo/Blue</material>
   </gazebo>
   <xacro:macro name="leg_material" params="side name">

File: src/hexa_description/urdf/hexapod.urdf.xacro (robot description, xacro)
@@ -66,10 +66,35 @@
   <xacro:property name="tibia_upper_rad"
                   value="${pi - geom['joints']['tibia']['lower_limit_deg'] * pi / 180}"/>
-  <!-- Body length and width are derived from the front and middle mounts
-       so the chassis always extends just past the hips: 10% margin per side. -->
+  <!-- Initial pose used by ros2_control's <initial_value>: same deg→rad
+       conversion as the <limit> window above. In sim, gz_ros2_control
+       applies it on spawn; on the real robot, the hardware plugin uses it
+       as the assumed pose for servos that cannot report position. Femur
+       and tibia are uniform across all six legs; the per-leg coxa value
+       lives inside the leg_joints_iface macro so it can apply the same
+       x/y mirror as mount_leg. -->
+  <xacro:property name="initial_femur_rad"
+                  value="${-geom['initial_pose']['femur']['above_horizontal_deg'] * pi / 180}"/>
+  <xacro:property name="initial_tibia_rad"
+                  value="${pi - geom['initial_pose']['tibia']['interior_deg'] * pi / 180}"/>
+  <!-- Body length and width are derived from the front and middle mounts.
+       Length extends 10% past the front hips; width is 80% of the middle
+       hip span, so the chassis is narrower than the coxa bases and the
+       middle bar (below) bridges the gap between them. -->
   <xacro:property name="body_length" value="${2 * geom['mounts']['l_front']['x']  * 1.1}"/>
-  <xacro:property name="body_width"  value="${2 * geom['mounts']['l_middle']['y'] * 1.1}"/>
-  <xacro:property name="body_height" value="${geom['body']['height']}"/>
-  <xacro:property name="body_mass"   value="${geom['body']['mass']}"/>
+  <xacro:property name="body_width"  value="${2 * geom['mounts']['l_middle']['y'] * 0.8}"/>
+  <!-- Body box vertical extent is split around the coxa joint plane
+       (= base_link origin, z=0). The box height is the sum of the two
+       halves; body_z_offset shifts the box origin so the coxa joints
+       end up at the requested z relative to the chassis (positive
+       offset moves the box centre up). Equal coxa_to_bottom and
+       coxa_to_top reproduce the previous centred-box behaviour. -->
+  <xacro:property name="coxa_to_bottom" value="${geom['body']['coxa_to_bottom']}"/>
+  <xacro:property name="coxa_to_top"    value="${geom['body']['coxa_to_top']}"/>
+  <xacro:property name="body_height"    value="${coxa_to_bottom + coxa_to_top}"/>
+  <xacro:property name="body_z_offset"  value="${(coxa_to_top - coxa_to_bottom) / 2}"/>
+  <xacro:property name="body_mass"      value="${geom['body']['mass']}"/>
+  <!-- Half-span between the middle coxa bases; the bar spans from
+       -middle_mount_y to +middle_mount_y along the body y-axis. -->
+  <xacro:property name="middle_mount_y" value="${geom['mounts']['l_middle']['y']}"/>
   <!-- =====================================================================
        Materials (just for colour in RViz / Gazebo).
@@ -102,7 +127,10 @@
          iyy = (1/12) m (x^2 + z^2)
          izz = (1/12) m (x^2 + y^2)
-       COM at link origin (the body box is centred on base_link). -->
-  <xacro:macro name="box_inertial" params="mass x y z">
+       COM defaults to the link origin; pass z_offset to shift it along
+       +z (used by base_link when the body box is split asymmetrically
+       around the coxa plane). -->
+  <xacro:macro name="box_inertial" params="mass x y z z_offset:=0">
     <inertial>
+      <origin xyz="0 0 ${z_offset}" rpy="0 0 0"/>
       <mass value="${mass}"/>
       <inertia ixx="${mass * (y*y + z*z) / 12.0}"
@@ -117,4 +145,5 @@
   <link name="base_link">
     <visual>
+      <origin xyz="0 0 ${body_z_offset}" rpy="0 0 0"/>
       <geometry>
         <box size="${body_length} ${body_width} ${body_height}"/>
@@ -123,4 +152,5 @@
     </visual>
     <collision>
+      <origin xyz="0 0 ${body_z_offset}" rpy="0 0 0"/>
       <geometry>
         <box size="${body_length} ${body_width} ${body_height}"/>
@@ -130,5 +160,37 @@
                         x="${body_length}"
                         y="${body_width}"
-                        z="${body_height}"/>
+                        z="${body_height}"
+                        z_offset="${body_z_offset}"/>
+  </link>
+  <!-- =====================================================================
+       Middle bar — decorative blue cylinder spanning the middle coxa
+       bases, with endcap spheres on each mount point. Lives in its own
+       link so the Gazebo material reference can paint it independently
+       of the dark-grey body box. Visual-only; the fixed joint lumps it
+       into base_link for dynamics, so no inertial entry is needed.
+       ===================================================================== -->
+  <joint name="middle_bar_joint" type="fixed">
+    <parent link="base_link"/>
+    <child  link="middle_bar"/>
+    <origin xyz="0 0 0" rpy="0 0 0"/>
+  </joint>
+  <link name="middle_bar">
+    <visual>
+      <origin xyz="0 0 0" rpy="${pi/2} 0 0"/>
+      <geometry>
+        <cylinder radius="${coxa_radius}" length="${2 * middle_mount_y}"/>
+      </geometry>
+      <material name="leg_blue"/>
+    </visual>
+    <visual>
+      <origin xyz="0 ${middle_mount_y} 0" rpy="0 0 0"/>
+      <geometry><sphere radius="${coxa_radius}"/></geometry>
+      <material name="leg_blue"/>
+    </visual>
+    <visual>
+      <origin xyz="0 ${-middle_mount_y} 0" rpy="0 0 0"/>
+      <geometry><sphere radius="${coxa_radius}"/></geometry>
+      <material name="leg_blue"/>
+    </visual>
   </link>
   <!-- =====================================================================
@@ -336,4 +398,16 @@
        ===================================================================== -->
   <xacro:macro name="leg_joints_iface" params="side name">
+    <!-- Per-leg coxa initial angle, derived from
+         initial_pose.coxa.l_{front,middle}_deg by the same x/y mirror as
+         mount_leg above:
+           - rear  : negate (front/rear mirror)
+           - r_*   : negate (left/right mirror)
+         Applying both leaves r_rear with the same sign as l_front. -->
+    <xacro:property name="ref_initial_coxa_deg"
+                    value="${geom['initial_pose']['coxa']['l_middle_deg' if name == 'middle' else 'l_front_deg']}"/>
+    <xacro:property name="initial_coxa_deg_after_fr"
+                    value="${-ref_initial_coxa_deg if name == 'rear' else ref_initial_coxa_deg}"/>
+    <xacro:property name="initial_coxa_rad"
+                    value="${(-initial_coxa_deg_after_fr if side == 'r' else initial_coxa_deg_after_fr) * pi / 180}"/>
     <joint name="${side}_${name}_coxa_joint">
       <command_interface name="position">
@@ -341,5 +415,7 @@
         <param name="max">${coxa_upper_rad}</param>
       </command_interface>
-      <state_interface name="position"/>
+      <state_interface name="position">
+        <param name="initial_value">${initial_coxa_rad}</param>
+      </state_interface>
       <state_interface name="velocity"/>
     </joint>
@@ -349,5 +425,7 @@
         <param name="max">${femur_upper_rad}</param>
       </command_interface>
-      <state_interface name="position"/>
+      <state_interface name="position">
+        <param name="initial_value">${initial_femur_rad}</param>
+      </state_interface>
       <state_interface name="velocity"/>
     </joint>
@@ -357,5 +435,7 @@
         <param name="max">${tibia_upper_rad}</param>
       </command_interface>
-      <state_interface name="position"/>
+      <state_interface name="position">
+        <param name="initial_value">${initial_tibia_rad}</param>
+      </state_interface>
       <state_interface name="velocity"/>
     </joint>

Commit message: feat: improve the velocity limiter

File: src/hexa_description/urdf/hexapod.gazebo.xacro (robot description, xacro)
@@ -38,4 +38,8 @@
        and the body doesn't slide. kp/kd are typical defaults for rigid
        contact at ~0.1 m foot scale.
+       The <sensor type="contact"> blocks emit gz.msgs.Contacts on
+       /contact/<foot> whenever the foot is touching another collider.
+       Each Contacts message carries world-frame contact points, which
+       the foot_paint dev node consumes to draw slip trails.
        =================================================================== -->
   <xacro:macro name="foot_contact" params="link">
@@ -45,4 +49,16 @@
       <kp>1.0e6</kp>
       <kd>10.0</kd>
+      <!-- The <topic> override is dropped because sdformat's URDF
+           converter ignores it; the sensor publishes on its default
+           /world/<world>/model/<model>/link/<link>/sensor/<sensor>/contact
+           name. ros_gz_bridge remaps it to /contact/<foot> via
+           hexa_simulation/config/contact_bridge.yaml. -->
+      <sensor name="${link}_contact" type="contact">
+        <update_rate>100</update_rate>
+        <always_on>true</always_on>
+        <contact>
+          <collision>${link}_collision</collision>
+        </contact>
+      </sensor>
     </gazebo>
   </xacro:macro>
@@ -53,4 +69,22 @@
   <xacro:foot_contact link="r_middle_foot"/>
   <xacro:foot_contact link="r_rear_foot"/>
+  <!-- ===================================================================
+       Preserve the foot-tibia fixed joints. sdformat-urdf lumps fixed
+       joints by default, which would merge each foot link into its
+       parent tibia and drop the per-link contact sensor declared above.
+       Keeping the joint preserves the foot as its own SDF link, so the
+       <gazebo reference="..._foot"> sensor block lands somewhere real.
+       =================================================================== -->
+  <xacro:macro name="preserve_foot_joint" params="joint">
+    <gazebo reference="${joint}">
+      <preserveFixedJoint>true</preserveFixedJoint>
+    </gazebo>
+  </xacro:macro>
+  <xacro:preserve_foot_joint joint="l_front_foot_joint"/>
+  <xacro:preserve_foot_joint joint="l_middle_foot_joint"/>
+  <xacro:preserve_foot_joint joint="l_rear_foot_joint"/>
+  <xacro:preserve_foot_joint joint="r_front_foot_joint"/>
+  <xacro:preserve_foot_joint joint="r_middle_foot_joint"/>
+  <xacro:preserve_foot_joint joint="r_rear_foot_joint"/>
   <!-- ===================================================================
        gz_ros2_control system plugin: hosts the ros2_control controller
