Commit message: feat: IMU + autoleveling

File: src/hexa_description/urdf/hexapod.gazebo.xacro (robot description, xacro)
@@ -87,4 +87,27 @@
   <xacro:preserve_foot_joint joint="r_rear_foot_joint"/>
   <!-- ===================================================================
+       IMU. Needs gz-sim-imu-system in the world; sim.launch.py bridges
+       the topic to /imu/data. Noise roughly an MPU6500 at a 41 Hz DLPF.
+       =================================================================== -->
+  <gazebo reference="imu_link">
+    <sensor name="imu" type="imu">
+      <always_on>true</always_on>
+      <update_rate>200</update_rate>
+      <topic>imu</topic>
+      <imu>
+        <angular_velocity>
+          <x><noise type="gaussian"><stddev>0.002</stddev></noise></x>
+          <y><noise type="gaussian"><stddev>0.002</stddev></noise></y>
+          <z><noise type="gaussian"><stddev>0.002</stddev></noise></z>
+        </angular_velocity>
+        <linear_acceleration>
+          <x><noise type="gaussian"><stddev>0.05</stddev></noise></x>
+          <y><noise type="gaussian"><stddev>0.05</stddev></noise></y>
+          <z><noise type="gaussian"><stddev>0.05</stddev></noise></z>
+        </linear_acceleration>
+      </imu>
+    </sensor>
+  </gazebo>
+  <!-- ===================================================================
        gz_ros2_control system plugin: hosts the ros2_control controller
        manager inside Gazebo and binds it to the <ros2_control> block in

File: src/hexa_description/urdf/hexapod.urdf.xacro (robot description, xacro)
@@ -167,4 +167,14 @@
   </link>
   <!-- =====================================================================
+       IMU frame. Axes aligned with base_link; the driver rotates the
+       sensor's own axes into it.
+       ===================================================================== -->
+  <joint name="imu_joint" type="fixed">
+    <parent link="base_link"/>
+    <child  link="imu_link"/>
+    <origin xyz="${geom['imu']['x']} ${geom['imu']['y']} ${geom['imu']['z']}" rpy="0 0 0"/>
+  </joint>
+  <link name="imu_link"/>
+  <!-- =====================================================================
        Middle bar — decorative blue cylinder spanning the middle coxa
        bases, with endcap spheres on each mount point. Lives in its own
